File: AxxSolder_hardware/AxxSolder.kicad_pcb (KiCad board)
At the start: 2 copper layers, 39 x 82.5 mm, 145 parts, among them IC1 TLV76733DRVR, IC2 OPA2387DSGT, IC3 LMR54406DBVR, IC4 STM32G431CBT6, IC5 TPD4E1U06DBVR, IC6 STUSB4500QTR, IC7 MAX16171ATA_VY+T, IC8 LTC4440AHMS8E, IC9 INA281A5QDBVRQ1, J1 USB4110-GF-A, J2 691243110009, J3 TSW-102-07-T-S, J4 61300611821, J5 TSW-102-07-T-S, J6 TSW-102-07-T-S, J7 TSW-108-07-T-S, Q1 STL9P3LLH6, Q2 STL10N3LLH5, Q3 2N7002NXAKR, U2 PEC11J-9215F-S0015, U3 BSC014N04LS

Commit message: Actualización Esquema y PCB
Parts:
- removed C31, C32: 10u, Capacitor_SMD:C_0603_1608Metric
- removed C33: 100n, Capacitor_SMD:C_0603_1608Metric
- removed D9: PMEG6020ER, footprints:PMEG6020ER115
- removed IC8: LTC4440AHMS8E, footprints:SOP65P490X110-9N
- removed R38: 4k7, Resistor_SMD:R_0603_1608Metric
- removed S1: ADTSM644RVTR, footprints:ADTSM644RVTR
- removed TP17: SW_TP, TestPoint:TestPoint_Pad_D1.0mm
- removed TP18: DIAG_TP, footprints:TSW-101-XX-YY-S
- removed U3: BSC014N04LS, footprints:BSC014N04LS
- added Q4: BSZ180P03NS3E, Package_TO_SOT_SMD:TDSON-8-1, B.Cu at (187.7, 81.1)
- added Q5: 2N7002NXAKR, footprints:SOT95P230X110-3N, B.Cu at (172.7, 80.8)
- added R49: 100, Resistor_SMD:R_0603_1608Metric, B.Cu at (179.8, 88.2)
- added R50: 4k7, Resistor_SMD:R_0603_1608Metric, B.Cu at (179.8, 86.4)
- added R51: 4k7, Resistor_SMD:R_1210_3225Metric_Pad1.30x2.65mm_HandSolder, B.Cu at (176.4, 81.1)
- added R52: 100, Resistor_SMD:R_0603_1608Metric, B.Cu at (179.8, 84.6)
- added U1: COS1415, Package_TO_SOT_SMD:SOT-23-5, B.Cu at (176.0, 89.2)
- IC2: footprint footprints:SON50P200X200X80-9N -> Package_SO:VSSOP-8_3x3mm_P0.65mm
- moved C30 7.16 mm to (178.9, 90.3), turned to 90 degrees
- moved J7 2.39 mm to (172.7, 123.9)
- moved IC2 0.93 mm to (180.8, 100.3)
- moved TP10 0.76 mm to (179.1, 103.0)
- moved C35 0.56 mm to (183.2, 75.8)
- moved D4 0.56 mm to (182.0, 79.8)
- moved C34 0.50 mm to (183.2, 77.4)
- moved R2 0.44 mm to (184.9, 100.6)
- moved R9 0.21 mm to (182.8, 97.8)
- moved TFT1 0.08 mm to (180.5, 126.6)
Connections:
- C30 pad 1: /RED -> GND
- C30 pad 2: /BOOST -> VDD
- J7 pad 1: +3.3V -> /SPI_CS
- J7 pad 2: GND -> /SPI_DC
- J7 pad 3: /SPI_SCK -> /SPI_RST
- J7 pad 4: unconnected-(J7-Pin_4-Pad4) -> /SPI_MOSI
- J7 pad 5: /SPI_MOSI -> /SPI_SCK
- J7 pad 6: /SPI_CS -> +3.3V
- J7 pad 7: /SPI_RST -> GND
- J7 pad 8: /SPI_DC -> /SD_CS
Routing:
- net VDD: track 58.8 -> 80.2 mm
- net Net-(Q5-G): track 0.00 -> 16.9 mm
- net GND: track 435.5 -> 451.9 mm, vias 167 -> 164
- net +7.5V: track 94.3 -> 79.1 mm
- net Net-(Q4-G): track 0.00 -> 14.5 mm
- net Net-(Q5-D): track 0.00 -> 13.6 mm
- net /BOOST: track 8.36 -> 0.00 mm
- net /RED: track 32.4 -> 24.2 mm
- net /SPI_DC: track 10.1 -> 18.2 mm, vias 0 -> 1
- net +3.3V: track 195.1 -> 202.4 mm, vias 16 -> 17
- net /SPI_CS: track 8.30 -> 14.9 mm, vias 0 -> 1
- net /SPI_SCK: track 14.3 -> 8.48 mm, vias 1 -> 0
- net /Heater: track 28.4 -> 24.9 mm, vias 1 -> 0
- net Net-(IC8-TG): track 2.85 -> 0.00 mm
- net Net-(IC2B-+): track 15.0 -> 17.8 mm
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- removed copper zone on B.Cu, net /BOOST
Other:
- board text added: "V3.2c"
- board text added: "V3.2c luicer"
- board text removed: "V3.1"
